File: kicad/all_mainboard/kicad.kicad_pcb (KiCad board)
At the start: 2 copper layers, 266 x 95 mm, 139 parts, among them J1 USB_A

Commit message: update pcb : move traces further from edges
Routing:
- net /tiny+ switch array standard/wr-2: track 287.1 -> 303.9 mm
- net /tiny+ switch array standard/r-7: track 115.0 -> 102.7 mm
- net /tiny+ switch array standard/wr-3: track 263.0 -> 273.4 mm
- net /tiny+ switch array standard/wr-0: track 336.9 -> 346.6 mm
- net /tiny+ switch array standard/wr-1: track 285.4 -> 294.6 mm
- net /tiny+ switch array standard/wr-4: track 260.2 -> 267.9 mm
- net /tiny+ switch array standard/r-2: track 148.6 -> 155.4 mm
- net /tiny+ switch array standard/r-3: track 133.7 -> 136.6 mm
- net /tiny+ switch array standard/r-4: track 114.1 -> 116.9 mm
- net Net-(D1-A+): track 101.2 -> 104.0 mm
- net Net-(D2-K-): track 73.9 -> 73.0 mm
- net Net-(A2-PadD4): track 21.0 -> 21.8 mm

Commit message: further pcb tweaks
Routing:
- net /tiny+ switch array standard/r-6: track 96.4 -> 97.1 mm
Changed lines of the file:
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@@
 	)
 	(segment
-		(start 106 74.5)
-		(end 104.5 73)
+		(start 106 75)
+		(end 104.5 73.5)
 		(width 0.2)
 		(layer "F.Cu")
@@
 	)
 	(segment
-		(start 106 68.5)
-		(end 106 55.5)
+		(start 110.18 100.5)
+		(end 110.18 97.96)
 		(width 0.2)
 		(layer "F.Cu")
@@
 	)
 	(segment
-		(start 104.5 73)
-		(end 104.5 70)
+		(start 98 36.5)
+		(end 98 32.07)
 		(width 0.2)
 		(layer "F.Cu")
@@
 	)
 	(segment
-		(start 106 40.5)
-		(end 103.5 38)
+		(start 107.5 89.5)
+		(end 106 88)
 		(width 0.2)
 		(layer "F.Cu")
@@
 	)
 	(segment
-		(start 98 36.5)
-		(end 98 32.07)
+		(start 104.5 73.5)
+		(end 104.5 70)
 		(width 0.2)
 		(layer "F.Cu")
@@
 	)
 	(segment
-		(start 110.18 100.5)
-		(end 110.18 97.96)
+		(start 106 49.5)
+		(end 106 40.5)
 		(width 0.2)
 		(layer "F.Cu")
@@
 	)
 	(segment
-		(start 106 88)
-		(end 106 74.5)
+		(start 107.5 95.28)
+		(end 107.5 89.5)
 		(width 0.2)
 		(layer "F.Cu")
@@
 	)
 	(segment
-		(start 104.5 51)
-		(end 106 49.5)
+		(start 104.5 54)
+		(end 104.5 51)
 		(width 0.2)
 		(layer "F.Cu")
@@
 	)
 	(segment
-		(start 103.5 38)
-		(end 99.5 38)
+		(start 99.5 38)
+		(end 98 36.5)
 		(width 0.2)
 		(layer "F.Cu")
@@
 	)
 	(segment
-		(start 110.18 97.96)
-		(end 107.5 95.28)
+		(start 106 88)
+		(end 106 75)
 		(width 0.2)
 		(layer "F.Cu")
@@
 	)
 	(segment
-		(start 106 55.5)
-		(end 104.5 54)
+		(start 106 68.5)
+		(end 106 55.5)
 		(width 0.2)
 		(layer "F.Cu")
@@
 	)
 	(segment
-		(start 106 49.5)
-		(end 106 40.5)
+		(start 106 55.5)
+		(end 104.5 54)
 		(width 0.2)
 		(layer "F.Cu")
@@
 	)
 	(segment
-		(start 107.5 89.5)
-		(end 106 88)
+		(start 103.5 38)
+		(end 99.5 38)
 		(width 0.2)
 		(layer "F.Cu")
@@
 	)
 	(segment
-		(start 99.5 38)
-		(end 98 36.5)
+		(start 106 40.5)
+		(end 103.5 38)
 		(width 0.2)
 		(layer "F.Cu")
@@
 	)
 	(segment
-		(start 104.5 70)
-		(end 106 68.5)
+		(start 104.5 51)
+		(end 106 49.5)
 		(width 0.2)
 		(layer "F.Cu")
@@
 	)
 	(segment
-		(start 107.5 95.28)
-		(end 107.5 89.5)
+		(start 104.5 70)
+		(end 106 68.5)
 		(width 0.2)
 		(layer "F.Cu")
@@
 	)
 	(segment
-		(start 104.5 54)
-		(end 104.5 51)
+		(start 110.18 97.96)
+		(end 107.5 95.28)
 		(width 0.2)
 		(layer "F.Cu")
@@
 	)
 	(segment
-		(start 132 99)
-		(end 130.5 100.5)
+		(start 132.5 92.5)
+		(end 132.5 96)
 		(width 0.2)
 		(layer "F.Cu")
@@
 	)
 	(segment
-		(start 132.839 72.41747)
-		(end 133 72.57847)
+		(start 132.799 48.201)
+		(end 133.69 47.31)
 		(width 0.2)
 		(layer "F.Cu")
@@
 	)
 	(segment
-		(start 132.799 48.201)
-		(end 133.69 47.31)
+		(start 132 99)
+		(end 130.5 100.5)
 		(width 0.2)
 		(layer "F.Cu")
@@
 	)
 	(segment
-		(start 133.69 82.92)
-		(end 132 84.61)
+		(start 133.69 47.31)
+		(end 133.69 44.92)
 		(width 0.2)
 		(layer "F.Cu")
@@
 	)
 	(segment
-		(start 133 64.61)
-		(end 133 71.26153)
+		(start 133.69 63.92)
+		(end 133.69 54.38847)
 		(width 0.2)
 		(layer "F.Cu")
@@
 	)
 	(segment
-		(start 133.69 47.31)
-		(end 133.69 44.92)
+		(start 132.5 96)
+		(end 132 96.5)
+		(width 0.2)
+		(layer "F.Cu")
+		(net "/tiny+ switch array standard/r-6")
+	)
+	(segment
+		(start 132 41)
+		(end 133.69 42.69)
 		(width 0.2)
 		(layer "F.Cu")
@@
 	(segment
 		(start 133.69 63.92)
-		(end 133.69 54.38847)
+		(end 132.5 65.11)
 		(width 0.2)
 		(layer "F.Cu")
@@
 	)
 	(segment
-		(start 132 41)
-		(end 133.69 42.69)
+		(start 132.5 84.11)
+		(end 132.5 89.5)
 		(width 0.2)
 		(layer "F.Cu")
@@
 	)
 	(segment
-		(start 133.69 42.69)
-		(end 133.69 44.92)
+		(start 133.69 80.69)
+		(end 133.69 82.92)
 		(width 0.2)
 		(layer "F.Cu")
@@
 	)
 	(segment
-		(start 133 71.26153)
-		(end 132.839 71.42253)
+		(start 133.69 42.69)
+		(end 133.69 44.92)
 		(width 0.2)
 		(layer "F.Cu")
@@
 	)
 	(segment
-		(start 133.69 80.69)
-		(end 133.69 82.92)
+		(start 132 92)
+		(end 132.5 92.5)
 		(width 0.2)
 		(layer "F.Cu")
@@
 	)
 	(segment
-		(start 133 80)
-		(end 133.69 80.69)
+		(start 134.19 27.81)
+		(end 132 30)
 		(width 0.2)
 		(layer "F.Cu")
@@
 	)
 	(segment
-		(start 134.19 27.81)
-		(end 132 30)
+		(start 132.5 79.5)
+		(end 133.69 80.69)
 		(width 0.2)
 		(layer "F.Cu")
@@
 	)
 	(segment
-		(start 133 72.57847)
-		(end 133 80)
+		(start 132 96.5)
+		(end 132 99)
 		(width 0.2)
 		(layer "F.Cu")
@@
 	)
 	(segment
-		(start 133.69 63.92)
-		(end 133 64.61)
+		(start 132.5 89.5)
+		(end 132 90)
 		(width 0.2)
 		(layer "F.Cu")
@@
 	)
 	(segment
-		(start 132.839 71.42253)
-		(end 132.839 72.41747)
+		(start 132 90)
+		(end 132 92)
 		(width 0.2)
 		(layer "F.Cu")
@@
 	)
 	(segment
-		(start 132 84.61)
-		(end 132 99)
+		(start 133.69 82.92)
+		(end 132.5 84.11)
 		(width 0.2)
 		(layer "F.Cu")
@@
 		(width 0.2)
 		(layer "F.Cu")
+		(net "/tiny+ switch array standard/r-6")
+	)
+	(segment
+		(start 132.5 65.11)
+		(end 132.5 79.5)
+		(width 0.2)
+		(layer "F.Cu")
